File: Dumper/Dumper.kicad_sch (KiCad schematic)
At the start: 0 parts

Commit message: Add Dumper circuit with two servos
Parts:
- added A1: Arduino_UNO_R3, Module:Arduino_UNO_R3, symbol MCU_Module:Arduino_UNO_R3
- added M1: Hatch Servo, symbol Motor:Motor_Servo
- added M2: Tube Rotation Servo, symbol Motor:Motor_Servo
Connections:
- new net: A1.25 (D10), M2.1 (PWM)
- new net: A1.5 (+5V), M1.2 (+), M2.2 (+)
- new net: A1.29 (GND), M1.3 (-), M2.3 (-)
- new net: A1.24 (D9), M1.1 (PWM)
- new net Earth: A1.6 (GND)
Changed lines of the file:
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@@
 (kicad_sch (version 20230121) (generator eeschema)
-  (paper "A4")
+  (paper "A5")
   (title_block
     (title "Dumper Simple Circuit")
     (date "2024-02-20")
   )
+  (junction (at 111.76 63.5) (diameter 0) (color 0 0 0 0)
+  )
+  (junction (at 109.22 77.47) (diameter 0) (color 0 0 0 0)
+  )
+  (wire (pts (xy 104.14 66.04) (xy 104.14 60.96))
+    (stroke (width 0) (type default))
+  )
+  (wire (pts (xy 109.22 77.47) (xy 121.92 77.47))
+    (stroke (width 0) (type default))
+  )
+  (wire (pts (xy 104.14 72.39) (xy 121.92 72.39))
+    (stroke (width 0) (type default))
+  )
+  (wire (pts (xy 109.22 66.04) (xy 121.92 66.04))
+    (stroke (width 0) (type default))
+  )
+  (wire (pts (xy 86.36 66.04) (xy 104.14 66.04))
+    (stroke (width 0) (type default))
+  )
+  (wire (pts (xy 104.14 60.96) (xy 121.92 60.96))
+    (stroke (width 0) (type default))
+  )
+  (wire (pts (xy 68.58 29.21) (xy 109.22 29.21))
+    (stroke (width 0) (type default))
+  )
+  (wire (pts (xy 73.66 86.36) (xy 73.66 93.98))
+    (stroke (width 0) (type default))
+  )
+  (wire (pts (xy 121.92 74.93) (xy 111.76 74.93))
+    (stroke (width 0) (type default))
+  )
+  (wire (pts (xy 76.2 87.63) (xy 76.2 86.36))
+    (stroke (width 0) (type default))
+  )
+  (wire (pts (xy 111.76 63.5) (xy 121.92 63.5))
+    (stroke (width 0) (type default))
+  )
+  (wire (pts (xy 111.76 74.93) (xy 111.76 63.5))
+    (stroke (width 0) (type default))
+  )
+  (wire (pts (xy 109.22 63.5) (xy 111.76 63.5))
+    (stroke (width 0) (type default))
+  )
+  (wire (pts (xy 104.14 68.58) (xy 104.14 72.39))
+    (stroke (width 0) (type default))
+  )
+  (wire (pts (xy 109.22 77.47) (xy 109.22 66.04))
+    (stroke (width 0) (type default))
+  )
+  (wire (pts (xy 76.2 87.63) (xy 109.22 87.63))
+    (stroke (width 0) (type default))
+  )
+  (wire (pts (xy 86.36 68.58) (xy 104.14 68.58))
+    (stroke (width 0) (type default))
+  )
+  (wire (pts (xy 68.58 33.02) (xy 68.58 29.21))
+    (stroke (width 0) (type default))
+  )
+  (wire (pts (xy 109.22 29.21) (xy 109.22 63.5))
+    (stroke (width 0) (type default))
+  )
+  (wire (pts (xy 109.22 87.63) (xy 109.22 77.47))
+    (stroke (width 0) (type default))
+  )
+  (symbol (lib_id "Motor:Motor_Servo") (at 129.54 74.93 0) (unit 1)
+    (in_bom yes) (on_board yes) (dnp no) (fields_autoplaced)
+    (property "Reference" "M2" (at 138.43 73.8616 0)
+      (effects (font (size 1.27 1.27)) (justify left))
+    )
+    (property "Value" "Tube Rotation Servo" (at 138.43 76.4016 0)
+      (effects (font (size 1.27 1.27)) (justify left))
+    )
+    (property "Footprint" "" (at 129.54 79.756 0)
+      (effects (font (size 1.27 1.27)) hide)
+    )
+    (property "Datasheet" "http://forums.parallax.com/uploads/attachments/46831/74481.png" (at 129.54 79.756 0)
+      (effects (font (size 1.27 1.27)) hide)
+    )
+    (pin "1")
+    (pin "2")
+    (pin "3")
+    (instances
+      (project "Dumper"
+        (path "/844fbdc4-262b-4967-a6a4-9afd0c766b74"
+          (reference "M2") (unit 1)
+        )
+      )
+    )
+  )
+  (symbol (lib_id "MCU_Module:Arduino_UNO_R3") (at 73.66 58.42 0) (mirror y) (unit 1)
+    (in_bom yes) (on_board yes) (dnp no)
+    (property "Reference" "A1" (at 66.6241 31.75 0)
+      (effects (font (size 1.27 1.27)) (justify left))
+    )
+    (property "Value" "Arduino_UNO_R3" (at 66.6241 34.29 0)
+      (effects (font (size 1.27 1.27)) (justify left))
+    )
+    (property "Footprint" "Module:Arduino_UNO_R3" (at 73.66 58.42 0)
+      (effects (font (size 1.27 1.27) italic) hide)
+    )
+    (property "Datasheet" "https://www.arduino.cc/en/Main/arduinoBoardUno" (at 73.66 58.42 0)
+      (effects (font (size 1.27 1.27)) hide)
+    )
+    (pin "1")
+    (pin "10")
+    (pin "11")
+    (pin "12")
+    (pin "13")
+    (pin "14")
+    (pin "15")
+    (pin "16")
+    (pin "17")
+    (pin "18")
+    (pin "19")
+    (pin "2")
+    (pin "20")
+    (pin "21")
+    (pin "22")
+    (pin "23")
+    (pin "24")
+    (pin "25")
+    (pin "26")
+    (pin "27")
+    (pin "28")
+    (pin "29")
+    (pin "3")
+    (pin "30")
+    (pin "31")
+    (pin "32")
+    (pin "4")
+    (pin "5")
+    (pin "6")
+    (pin "7")
+    (pin "8")
+    (pin "9")
+    (instances
+      (project "Dumper"
+        (path "/844fbdc4-262b-4967-a6a4-9afd0c766b74"
+          (reference "A1") (unit 1)
+        )
+      )
+    )
+  )
+  (symbol (lib_id "Motor:Motor_Servo") (at 129.54 63.5 0) (unit 1)
+    (in_bom yes) (on_board yes) (dnp no) (fields_autoplaced)
+    (property "Reference" "M1" (at 138.43 62.4316 0)
+      (effects (font (size 1.27 1.27)) (justify left))
+    )
+    (property "Value" "Hatch Servo" (at 138.43 64.9716 0)
+      (effects (font (size 1.27 1.27)) (justify left))
+    )
+    (property "Footprint" "" (at 129.54 68.326 0)
+      (effects (font (size 1.27 1.27)) hide)
+    )
+    (property "Datasheet" "http://forums.parallax.com/uploads/attachments/46831/74481.png" (at 129.54 68.326 0)
+      (effects (font (size 1.27 1.27)) hide)
+    )
+    (pin "1")
+    (pin "2")
+    (pin "3")
+    (instances
+      (project "Dumper"
+        (path "/844fbdc4-262b-4967-a6a4-9afd0c766b74"
+          (reference "M1") (unit 1)
+        )
+      )
+    )
+  )
+  (symbol (lib_id "power:Earth") (at 73.66 93.98 0) (unit 1)
+    (in_bom yes) (on_board yes) (dnp no) (fields_autoplaced)
+    (property "Reference" "#PWR01" (at 73.66 100.33 0)
+      (effects (font (size 1.27 1.27)) hide)
+    )
+    (property "Value" "Earth" (at 73.66 97.79 0)
+      (effects (font (size 1.27 1.27)) hide)
+    )
+    (property "Footprint" "" (at 73.66 93.98 0)
+      (effects (font (size 1.27 1.27)) hide)
+    )
+    (property "Datasheet" "~" (at 73.66 93.98 0)
+      (effects (font (size 1.27 1.27)) hide)
+    )
+    (pin "1")
+    (instances
+      (project "Dumper"
+        (path "/844fbdc4-262b-4967-a6a4-9afd0c766b74"
+          (reference "#PWR01") (unit 1)
+        )
+      )
+    )
+  )
   (sheet_instances
